File: IrrationaLink.kicad_pcb (KiCad board)
At the start: 2 copper layers, 35 x 24 mm, 38 parts, among them J1 USB_C_Receptacle_USB2.0, J2 Conn_02x05_Odd_Even, J3 Conn_02x05_Odd_Even, SW1 SW_Push, U1 ESP32-C3, U2 LM2937xMP, Y1 ABM11W-40.0000MHZ-8-B1U-T3

Commit message: Connect all shield pads
Routing:
- net /SHIELD: track 11.7 -> 24.4 mm
Changed lines of the file:
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@@
   (segment (start 152.58 76.2) (end 152.58 77.585) (width 0.4) (layer "F.Cu") (net 22))
   (segment (start 152.58 77.585) (end 152.675 77.68) (width 0.4) (layer "F.Cu") (net 22))
+  (segment (start 148.495 77.105) (end 149.727 75.873) (width 1) (layer "B.Cu") (net 22))
+  (segment (start 151.383976 75.873) (end 152.675 77.164024) (width 1) (layer "B.Cu") (net 22))
+  (segment (start 148.495 86.32) (end 148.495 86.895) (width 1) (layer "B.Cu") (net 22))
+  (segment (start 149.727 75.873) (end 151.383976 75.873) (width 1) (layer "B.Cu") (net 22))
+  (segment (start 149.727 88.127) (end 151.473 88.127) (width 1) (layer "B.Cu") (net 22))
+  (segment (start 152.675 77.164024) (end 152.675 77.68) (width 1) (layer "B.Cu") (net 22))
+  (segment (start 148.495 86.895) (end 149.727 88.127) (width 1) (layer "B.Cu") (net 22))
   (segment (start 152.675 86.32) (end 152.675 77.68) (width 1) (layer "B.Cu") (net 22))
+  (segment (start 148.495 77.68) (end 148.495 77.105) (width 1) (layer "B.Cu") (net 22))
+  (segment (start 152.675 86.925) (end 152.675 86.32) (width 1) (layer "B.Cu") (net 22))
+  (segment (start 151.473 88.127) (end 152.675 86.925) (width 1) (layer "B.Cu") (net 22))
   (segment (start 133.584852 87.384852) (end 133.584852 86.1974) (width 0.25) (layer "F.Cu") (net 23))
   (segment (start 133.8 88.7) (end 133.8 87.6) (width 0.25) (layer "F.Cu") (net 23))

Commit message: Add via stitching
Routing:
- net GND: vias 48 -> 76
Changed lines of the file:
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@@
   (segment (start 132.1 88.3) (end 132.1 88.28) (width 0.4) (layer "F.Cu") (net 7))
   (segment (start 138.8 79.375) (end 137.575 79.375) (width 0.4) (layer "F.Cu") (net 7))
+  (via (at 129.945 92.759999) (size 0.4) (drill 0.3) (layers "F.Cu" "B.Cu") (free) (net 7))
   (via (at 130.4 81.2) (size 0.4) (drill 0.3) (layers "F.Cu" "B.Cu") (free) (net 7))
   (via (at 128.8 80.3) (size 0.4) (drill 0.3) (layers "F.Cu" "B.Cu") (free) (net 7))
   (via (at 126.9 82.7) (size 0.4) (drill 0.3) (layers "F.Cu" "B.Cu") (free) (net 7))
+  (via (at 132.485 72.439999) (size 0.4) (drill 0.3) (layers "F.Cu" "B.Cu") (free) (net 7))
+  (via (at 124.865 72.439999) (size 0.4) (drill 0.3) (layers "F.Cu" "B.Cu") (free) (net 7))
+  (via (at 124.865 87.679999) (size 0.4) (drill 0.3) (layers "F.Cu" "B.Cu") (free) (net 7))
   (via (at 129.8 81.2) (size 0.4) (drill 0.3) (layers "F.Cu" "B.Cu") (free) (net 7))
   (via (at 143.2 81.2035) (size 0.9) (drill 0.4) (layers "F.Cu" "B.Cu") (free) (net 7))
+  (via (at 127.405 80.059999) (size 0.4) (drill 0.3) (layers "F.Cu" "B.Cu") (free) (net 7))
+  (via (at 122.325 87.679999) (size 0.4) (drill 0.3) (layers "F.Cu" "B.Cu") (free) (net 7))
+  (via (at 137.565 77.519999) (size 0.4) (drill 0.3) (layers "F.Cu" "B.Cu") (free) (net 7))
   (via (at 141.2 83.2) (size 0.9) (drill 0.4) (layers "F.Cu" "B.Cu") (free) (net 7))
   (via (at 128.1 82.7) (size 0.4) (drill 0.3) (layers "F.Cu" "B.Cu") (free) (net 7))
+  (via (at 152.805 74.979999) (size 0.4) (drill 0.3) (layers "F.Cu" "B.Cu") (free) (net 7))
+  (via (at 150.265 92.759999) (size 0.4) (drill 0.3) (layers "F.Cu" "B.Cu") (free) (net 7))
   (via (at 141.2 81.2035) (size 0.9) (drill 0.4) (layers "F.Cu" "B.Cu") (free) (net 7))
   (via (at 146.7 77.3) (size 0.9) (drill 0.4) (layers "F.Cu" "B.Cu") (free) (net 7))
@@
   (via (at 134.2 78.4) (size 0.4) (drill 0.3) (layers "F.Cu" "B.Cu") (free) (net 7))
   (via (at 132.834851 83.7487) (size 0.4) (drill 0.3) (layers "F.Cu" "B.Cu") (net 7))
+  (via (at 124.865 92.759999) (size 0.4) (drill 0.3) (layers "F.Cu" "B.Cu") (free) (net 7))
+  (via (at 140.105 85.139999) (size 0.4) (drill 0.3) (layers "F.Cu" "B.Cu") (free) (net 7))
   (via (at 145.2 83.2) (size 0.9) (drill 0.4) (layers "F.Cu" "B.Cu") (free) (net 7))
+  (via (at 122.325 74.979999) (size 0.4) (drill 0.3) (layers "F.Cu" "B.Cu") (free) (net 7))
   (via (at 131.834851 84.7487) (size 0.4) (drill 0.3) (layers "F.Cu" "B.Cu") (net 7))
   (via (at 127.5 82.7) (size 0.4) (drill 0.3) (layers "F.Cu" "B.Cu") (free) (net 7))
+  (via (at 119.785 74.979999) (size 0.4) (drill 0.3) (layers "F.Cu" "B.Cu") (free) (net 7))
   (via (at 131.834851 83.7487) (size 0.4) (drill 0.3) (layers "F.Cu" "B.Cu") (net 7))
   (via (at 132.834851 82.7487) (size 0.4) (drill 0.3) (layers "F.Cu" "B.Cu") (net 7))
+  (via (at 129.945 74.979999) (size 0.4) (drill 0.3) (layers "F.Cu" "B.Cu") (free) (net 7))
   (via (at 130.6 76) (size 0.4) (drill 0.3) (layers "F.Cu" "B.Cu") (free) (net 7))
   (via (at 137.2 87) (size 0.4) (drill 0.3) (layers "F.Cu" "B.Cu") (net 7))
   (via (at 126.2 91.5) (size 0.9) (drill 0.4) (layers "F.Cu" "B.Cu") (net 7))
+  (via (at 132.485 74.979999) (size 0.4) (drill 0.3) (layers "F.Cu" "B.Cu") (free) (net 7))
   (via (at 128.799503 85) (size 0.4) (drill 0.3) (layers "F.Cu" "B.Cu") (free) (net 7))
   (via (at 145.2 81.2035) (size 0.9) (drill 0.4) (layers "F.Cu" "B.Cu") (free) (net 7))
@@
   (via (at 131.834851 82.7487) (size 0.4) (drill 0.3) (layers "F.Cu" "B.Cu") (net 7))
   (via (at 127.1 81.2) (size 0.4) (drill 0.3) (layers "F.Cu" "B.Cu") (free) (net 7))
+  (via (at 152.805 72.439999) (size 0.4) (drill 0.3) (layers "F.Cu" "B.Cu") (free) (net 7))
   (via (at 128.7 82.7) (size 0.4) (drill 0.3) (layers "F.Cu" "B.Cu") (free) (net 7))
+  (via (at 152.805 90.219999) (size 0.4) (drill 0.3) (layers "F.Cu" "B.Cu") (free) (net 7))
   (via (at 143.2 83.2) (size 0.9) (drill 0.4) (layers "F.Cu" "B.Cu") (free) (net 7))
   (via (at 150.9 83.999999) (size 0.9) (drill 0.4) (layers "F.Cu" "B.Cu") (free) (net 7))
@@
   (via (at 146.6 85.2) (size 0.9) (drill 0.4) (layers "F.Cu" "B.Cu") (free) (net 7))
   (via (at 125.7 82.7) (size 0.4) (drill 0.3) (layers "F.Cu" "B.Cu") (free) (net 7))
+  (via (at 119.785 90.219999) (size 0.4) (drill 0.3) (layers "F.Cu" "B.Cu") (free) (net 7))
   (via (at 128.2 85) (size 0.4) (drill 0.3) (layers "F.Cu" "B.Cu") (free) (net 7))
   (via (at 129.3 82.7) (size 0.4) (drill 0.3) (layers "F.Cu" "B.Cu") (free) (net 7))
   (via (at 137.5 79.3) (size 0.9) (drill 0.4) (layers "F.Cu" "B.Cu") (net 7))
+  (via (at 137.565 82.599999) (size 0.4) (drill 0.3) (layers "F.Cu" "B.Cu") (free) (net 7))
+  (via (at 127.405 72.439999) (size 0.4) (drill 0.3) (layers "F.Cu" "B.Cu") (free) (net 7))
   (via (at 126.3 80.2) (size 0.4) (drill 0.3) (layers "F.Cu" "B.Cu") (free) (net 7))
   (via (at 133.834851 82.7487) (size 0.4) (drill 0.3) (layers "F.Cu" "B.Cu") (net 7))
   (via (at 126.3 82.7) (size 0.4) (drill 0.3) (layers "F.Cu" "B.Cu") (free) (net 7))
+  (via (at 119.785 72.439999) (size 0.4) (drill 0.3) (layers "F.Cu" "B.Cu") (free) (net 7))
   (via (at 125.5 81.2) (size 0.4) (drill 0.3) (layers "F.Cu" "B.Cu") (free) (net 7))
   (via (at 131.7 88.7) (size 0.4) (drill 0.3) (layers "F.Cu" "B.Cu") (free) (net 7))
   (via (at 151 76.8) (size 0.6) (drill 0.3) (layers "F.Cu" "B.Cu") (net 7))
+  (via (at 127.405 77.519999) (size 0.4) (drill 0.3) (layers "F.Cu" "B.Cu") (free) (net 7))
+  (via (at 119.785 87.679999) (size 0.4) (drill 0.3) (layers "F.Cu" "B.Cu") (free) (net 7))
   (via (at 127.7 81.2) (size 0.4) (drill 0.3) (layers "F.Cu" "B.Cu") (free) (net 7))
+  (via (at 127.405 74.979999) (size 0.4) (drill 0.3) (layers "F.Cu" "B.Cu") (free) (net 7))
   (via (at 128.3 81.2) (size 0.4) (drill 0.3) (layers "F.Cu" "B.Cu") (free) (net 7))
   (via (at 127.8 86.5) (size 0.6) (drill 0.3) (layers "F.Cu" "B.Cu") (free) (net 7))
+  (via (at 124.865 90.219999) (size 0.4) (drill 0.3) (layers "F.Cu" "B.Cu") (free) (net 7))
+  (via (at 122.325 92.759999) (size 0.4) (drill 0.3) (layers "F.Cu" "B.Cu") (free) (net 7))
+  (via (at 124.865 74.979999) (size 0.4) (drill 0.3) (layers "F.Cu" "B.Cu") (free) (net 7))
   (via (at 151 87.2) (size 0.6) (drill 0.3) (layers "F.Cu" "B.Cu") (net 7))
+  (via (at 132.485 92.759999) (size 0.4) (drill 0.3) (layers "F.Cu" "B.Cu") (free) (net 7))
   (segment (start 139.03 74.4) (end 141.93 77.3) (width 1) (layer "B.Cu") (net 7))
   (segment (start 139.03 92.18) (end 139.03 89.64) (width 1) (layer "B.Cu") (net 7))
@@
     )
   )
+  (group "ViaStitching GND" (id f6741f10-91dc-4dcf-812e-8999337b9c31)
+    (members
+      096b7cac-884c-4e98-9d45-9dafc5276c7c
+      0fd1274b-2bad-4aa3-b869-e1b07068dff1
+      1073b655-5fcc-4a18-b5c1-ef005caae657
+      19550cdb-5ab4-4234-94a3-4f83afa39ecd
+      1ff1773c-a0c2-4d58-a5ed-9ade299ef146
+      224b1bbf-3c61-42d1-900e-80d6b6479d5c
+      22b2ab33-8fa9-4c02-948d-7f47a39055c4
+      2f328f85-b913-41c7-8831-9630bc6a74ef
+      34e42586-121c-4094-913b-98f63cf75c10
+      44f0a022-e033-49e6-93fa-5fe4dd53cbfb
+      45ecd074-0b52-4790-9e86-b3bfc4bb36a5
+      46292b03-760b-49ce-b317-8cdecba956e9
+      4c60c335-769a-458a-a1c6-a0cc07df772d
+      5fadd70c-944d-41f8-85e4-800a026dcc11
+      6f0c32d6-2320-4c4a-b3c6-39598d63ddb8
+      8ecb57b5-20b8-4426-85b0-6287f9360761
+      9434e165-b802-42ad-83e6-4530e8d7010e
+      bd1c057a-e0cd-4b1f-a759-c75163face20
+      c69e40d5-8245-4c18-83d9-961d727baa05
+      c6b93f14-29f4-42dd-b72a-1541588149c0
+      d62bfd07-4736-4524-9650-672ae659cc12
+      de9f017c-826f-425a-b923-f7c8cbf0d932
+      e01bcc30-2eff-4c05-904c-abaeb615d6f6
+      e6cb9112-d52f-4ae5-9da3-36328de2ba5f
+      ee1e415a-fd59-4631-9f1b-6a49071b5051
+      ee6d68a9-de93-4e5c-9d14-cdcd36f4bb9b
+      f7c6ba59-c602-43d3-8d16-65613cc86614
+      fdcb63cc-41cb-4d20-b77a-8a238ad61ab1
+    )
+  )
